File: pcb/pss_mcu_pcb/pss_mcu_pcb.kicad_pcb (KiCad board)
At the start: 4 copper layers, 30.1 x 47.4 mm, 50 parts, among them J1 STM32_Prog, J2 UART_Prog, J3 Conn_01x18, J4 Conn_01x18, SW1 Boot, SW2 EN, SW3 SW_Push, U1 LM3940IMP-3.3_NOPB, U2 LM358, U3 STM32F030K6Tx, U4 ESP32-WROOM-32U

Commit message: Change resistor value
Parts:
- R13: value 7.5 -> 100
